File: oneDpong.brd (EAGLE design)
At the start: 136.4 x 80 mm, 66 parts, among them IC1 MEGA8-AI, IC2 74HC257D, IC3 LM386M-1, IC4 NPIC6C596, IC5 NPIC6C596

Commit message: tweaks
Parts:
- moved PWR 0.25 mm to (123.2, 36.3)
Changed lines of the file:
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@@
 <setting verticaltext="up"/>
 </settings>
-<grid distance="2" unitdist="mil" unit="mil" style="lines" multiple="1" display="yes" altdistance="0.005" altunitdist="inch" altunit="inch"/>
+<grid distance="0.05" unitdist="inch" unit="inch" style="lines" multiple="1" display="yes" altdistance="0.005" altunitdist="inch" altunit="inch"/>
 <layers>
 <layer number="1" name="Top" color="4" fill="1" visible="yes" active="yes"/>
@@
 <attribute name="MF" value="" x="79.375" y="26.543" size="1.778" layer="28" rot="MR180" display="off"/>
 <attribute name="OC_FARNELL" value="9171371" x="79.375" y="26.543" size="1.778" layer="28" rot="MR180" display="off"/>
-<attribute name="NAME" x="73.0504" y="23.114" size="1.27" layer="26" rot="MR180"/>
+<attribute name="NAME" x="71.6534" y="22.987" size="1.27" layer="26" rot="MR180"/>
 </element>
 <element name="C3" library="rcl" package="C0805" value="" x="66.04" y="35.56" smashed="yes" rot="MR0">
@@
 <attribute name="VALUE" x="129.54" y="13.335" size="1.27" layer="28" rot="MR0"/>
 </element>
-<element name="PWR" library="adafruit" package="LED3MM" value="" x="123.19" y="36.068" smashed="yes" rot="MR180">
-<attribute name="NAME" x="121.031" y="39.878" size="1.27" layer="26" ratio="10" rot="MR180"/>
-<attribute name="VALUE" x="125.095" y="37.719" size="1.27" layer="28" ratio="10" rot="MR180"/>
+<element name="PWR" library="adafruit" package="LED3MM" value="" x="123.19" y="36.322" smashed="yes" rot="MR180">
+<attribute name="NAME" x="121.031" y="40.132" size="1.27" layer="26" ratio="10" rot="MR180"/>
+<attribute name="VALUE" x="125.095" y="37.973" size="1.27" layer="28" ratio="10" rot="MR180"/>
 </element>
 <element name="R17" library="rcl" package="R0805" value="" x="121.92" y="31.75" smashed="yes" rot="MR270">
@@
 <contactref element="R17" pad="1"/>
 <contactref element="PWR" pad="A"/>
-<wire x1="121.92" y1="32.7" x2="121.92" y2="36.068" width="0.4064" layer="16"/>
+<wire x1="121.92" y1="32.7" x2="121.92" y2="36.322" width="0.4064" layer="16"/>
 </signal>
 <signal name="N$27">
