File: oneDpong.brd (EAGLE design)
At the start: 136.4 x 80 mm, 71 parts, among them IC1 MEGA8-AI, IC2 74HC257D, IC3 LM386M-1, IC4 NPIC6C596, IC5 NPIC6C596, IC6 NCP361SNT1G, Q2 NTD5867NL_NMOSFET

Commit message: V3 BOARD
Parts:
- removed R22: 100r, rcl:R0805
- removed TP2: TPB2,54, testpad:B2,54
- added R19: 1k, rcl:R0805
- added TP1: TPB1,27, testpad:B1,27
- added X1: (no value), crystal:HC49U-V
- C10: value (none) -> 47n
- C11: value 100n -> (none)
- C12, C13: value (none) -> 100n; device rcl:E2,5-6 -> rcl:C0805
- C14: value 1u -> (none)
- C15: value (none) -> 1u
- C4: device rcl:C0805 -> rcl:E2,5-6
- C7: value 47n -> (none)
- C9: value 100n -> (none); device rcl:C0805 -> rcl:E2,5-6
- IC1: value MEGA8-AI -> NPIC6C596; device atmel:TQFP32-08 -> jasons_stuff:SO16
- IC3: value LM386M-1 -> MEGA8-AI; device linear:SO08 -> atmel:TQFP32-08
- IC4: value NPIC6C596 -> LM386M-1; device jasons_stuff:SO16 -> linear:SO08
- Q1: value (none) -> SPD30P06PTO252; device crystal:HC49U-V -> transistor-fet:TO252
- Q2: value NTD5867NL_NMOSFET -> (none); device jason_eagle6:DPACK -> transistor:SOT23-BEC
- R10: value 10r -> 100r
- R11: value 1k -> 100r
- R13: value 100r -> 10r
- R14, R15, R7: value 100r -> (none)
- R16, R17, R18, R9: value (none) -> 100r
- R21: value 1k -> (none)
- R6: value 100r -> 1k
- moved C15 112.6 mm to (45.7, 22.9), turned to 180 degrees
- moved C1 96.7 mm to (143.5, 78.7)
- moved R14 91.1 mm to (39.4, 74.9)
- moved R13 85.2 mm to (47.0, 73.7), turned to 270 degrees
- moved R15 81.8 mm to (45.7, 62.2), turned to 90 degrees
- moved R5 76.5 mm to (118.1, 24.1), turned to 0 degrees
- moved R2 71.1 mm to (118.1, 31.8), turned to 0 degrees
- moved C13 63.4 mm to (43.2, 63.5), turned to 90 degrees
- moved IC4 62.9 mm to (49.5, 68.6), turned to 90 degrees
- moved IC3 51.6 mm to (79.4, 26.5), turned to 180 degrees
- moved R1 47.7 mm to (118.1, 34.4), turned to 180 degrees
- moved R8 46.5 mm to (82.5, 57.1)
- moved R4 44.7 mm to (118.1, 26.7), turned to 0 degrees
- moved R18 44.5 mm to (41.9, 30.5), turned to 90 degrees
- moved R12 43.7 mm to (74.9, 38.2), turned to 90 degrees
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Connections:
- removed net N$32: 5VA4.1, Q2.2
- removed net Z: Q2.1, R20.1, R21.2
- new net N$13: 5VA2.1, Q1.3
- new net N$29: Q1.1, Q2.C, R20.2
- new net N$30: Q2.B, R19.1
- net COL0: now also R9.2; no longer R6.2
- net COL1: now also R8.2; no longer R7.2
- net COL2: now also R18.2; no longer R5.2
- net COL3: now also R17.2; no longer R8.2
- net COL4: now also R16.2; no longer R2.2
- net COL5: now also R12.2; no longer R4.2
- net COL6: now also R10.2; no longer R1.2
- net COL7: now also R11.2; no longer R3.2
- net DISP0: now also IC3.12, R9.1; no longer IC1.12, R6.1
- net DISP1: now also IC3.13, R8.1; no longer IC1.13, R7.1
- net DISP2: now also IC3.32, R18.1; no longer IC1.32, R5.1
- net DISP3: now also IC3.1, R17.1; no longer IC1.1, R8.1
- net DISP4: now also IC3.2, R16.1; no longer IC1.2, R2.1
- net DISP5: now also IC3.9, R12.1; no longer IC1.9, R4.1
- net DISP6: now also IC3.10, R10.1; no longer IC1.10, R1.1
- net DISP7: now also IC3.11, R11.1; no longer IC1.11, R3.1
- net DISP_DS: now also IC3.23; no longer IC1.23
- net DISP_DS2: now also IC1.2; no longer IC4.2
- net DISP_SHCP: now also IC1.15, IC3.24; no longer IC1.24, IC4.15
- net DISP_STCP: now also IC1.10, IC3.25; no longer IC1.25, IC4.10
- net ENA_STRIP: now also IC3.14, R19.2, TP1.TP; no longer IC1.14, R21.1, TP2.TP
- net GND: now also 5VA4.1, C12.1, C15.2, C4.-, C7.1, C9.-, IC1.16, IC1.8, IC3.21, IC3.3, IC3.5, IC4.2, IC4.4, Q2.E, R1.2, R13.2, R6.1; no longer C1.2, C12.-, C13.-, C4.1, C9.1, IC1.21, IC1.3, IC1.5, IC3.2, IC3.4, IC4.16, IC4.8, Q2.3, R10.2, R11.1, R20.2, R22.2
- net MISO: now also IC3.16; no longer IC1.16
- net MOSI2: now also R4.1; no longer R13.1
- net N$1: now also IC3.30; no longer IC1.30
- net N$10: now also R3.2; no longer R14.2
- net N$11: now also R5.2; no longer R15.2
- net N$12: now also R2.1; no longer R12.1
- net N$14: now also IC3.31; no longer IC1.31
- net N$15: now also R5.1; no longer R15.1
- net N$16: now also R14.2; no longer R18.2
- net N$17: now also IC4.3; no longer IC3.3
- net N$18: now also IC3.28; no longer IC1.28
- net N$19: now also C10.2, IC4.5; no longer C7.2, IC3.5
- net N$2: now also R1.1; no longer R22.1
- net N$21: now also C12.2, IC4.7; no longer C9.2, IC3.7
- net N$22: now also IC4.1, R15.2; no longer IC3.1, R16.2
- net N$23: now also C11.2, R15.1; no longer C10.2, R16.1
- net N$24: now also C11.1, IC4.8; no longer C10.1, IC3.8
- net N$25: now also C13.2, R14.1; no longer C11.2, R18.1
- net N$26: now also R21.1; no longer R17.1
- net N$27: now also R6.2; no longer R11.2
- net N$3: now also C7.2, IC3.7, X1.2; no longer C3.2, IC1.7, Q1.2
- net N$4: now also C6.2, IC3.8, X1.1; no longer C4.2, IC1.8, Q1.1
- net N$5: now also R2.2; no longer R12.2
- net N$6: now also R4.2; no longer R13.2
- net N$7: now also IC3.17; no longer IC1.17
- net N$8: now also C10.1, R13.1; no longer C7.1, R10.1
- net N$9: now also C1.2; no longer C15.2
- net PMOSI: now also IC3.15; no longer IC1.15
- net Q0A1: now also IC1.3; no longer IC4.3
- net Q1A1: now also IC1.4; no longer IC4.4
- net Q2A1: now also IC1.5; no longer IC4.5
- net Q3A1: now also IC1.6; no longer IC4.6
- net Q4A1: now also IC1.11; no longer IC4.11
- net Q5A1: now also IC1.12; no longer IC4.12
- net Q6A1: now also IC1.13; no longer IC4.13
- net Q7A1: now also IC1.14; no longer IC4.14
- net RESET: now also C1.1, IC3.29, R7.1; no longer C15.1, IC1.29, R9.1
- net SCK1: now also R3.1; no longer R14.1
- net SOUND: now also C13.1, IC3.26; no longer C11.1, IC1.26
- net SW1: now also IC3.27; no longer IC1.27
- net VCC: now also C14.1, C15.1, C3.2, C4.+, C9.+, IC1.1, IC1.7, IC3.18, IC3.20, IC3.4, IC4.6, R21.2, R7.2; no longer C1.1, C12.+, C13.+, C16.1, C6.2, IC1.18, IC1.20, IC1.4, IC1.6, IC4.1, IC4.7, R17.2, R9.2
- net VIN: now also C16.1, Q1.2, R20.1; no longer 5VA2.1, C14.1
Routing:
- net VIN: track 44.6 -> 19.3 mm
- net N$32: track 11.5 -> 0.00 mm
- net N$28: track 16.0 -> 5.52 mm
- net N$13: track 0.00 -> 8.71 mm
- net GND: track 146.1 -> 137.4 mm
- net N$29: track 0.00 -> 7.38 mm
- net Z: track 6.34 -> 0.00 mm
- net N$30: track 0.00 -> 3.07 mm
Other:
- board text removed: "GND"
