File: oneDpong.sch (EAGLE design)
At the start: 66 parts, among them IC1 MEGA8-AI, IC2 74HC257D, IC3 LM386M-1, IC4 NPIC6C596, IC5 NPIC6C596

Commit message: stuff
Parts:
- removed C14: (no value), rcl:C-EUC0805
- removed GND1, GND2, VCC1, VCC2: (no value), pinhead:PINHD-1X1
- added C15: (no value), rcl:C-EUC0805
- added R18: (no value), rcl:R-EU_R0805
Connections:
- new net N$25: C11.2, R18.1
- new net N$9: C15.2, JP1.1
- net GND: no longer GND1.1, GND2.1
- net N$16: now also R18.2; no longer C11.2
- net RESET: now also C15.1, IC1.PC6(/RESET), R9.1; no longer C14.2, JP1.1
- net RST0: no longer C14.1, IC1.PC6(/RESET), R9.1
- net VCC: no longer VCC1.1, VCC2.1
Other:
- moved on the sheet: C11
Changed lines of the file:
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@@
 <part name="SW_GND1" library="pinhead" deviceset="PINHD-1X1" device=""/>
 <part name="SW_GND2" library="pinhead" deviceset="PINHD-1X1" device=""/>
-<part name="VCC1" library="pinhead" deviceset="PINHD-1X1" device=""/>
-<part name="VCC2" library="pinhead" deviceset="PINHD-1X1" device=""/>
-<part name="GND1" library="pinhead" deviceset="PINHD-1X1" device=""/>
-<part name="GND2" library="pinhead" deviceset="PINHD-1X1" device=""/>
 <part name="RST" library="pinhead" deviceset="PINHD-1X1" device=""/>
 <part name="RST_GND" library="pinhead" deviceset="PINHD-1X1" device=""/>
-<part name="C14" library="rcl" deviceset="C-EU" device="C0805"/>
 <part name="P2GND" library="pinhead" deviceset="PINHD-1X1" device=""/>
 <part name="P1GND" library="pinhead" deviceset="PINHD-1X1" device=""/>
 <part name="R10" library="rcl" deviceset="R-EU_" device="R0805"/>
+<part name="C15" library="rcl" deviceset="C-EU" device="C0805"/>
+<part name="R18" library="rcl" deviceset="R-EU_" device="R0805"/>
 </parts>
 <sheets>
@@
 <instance part="C10" gate="G$1" x="320.04" y="-55.88" rot="R180"/>
 <instance part="R16" gate="G$1" x="314.96" y="-55.88" rot="R270"/>
-<instance part="C11" gate="G$1" x="281.94" y="-50.8"/>
+<instance part="C11" gate="G$1" x="281.94" y="-35.56"/>
 <instance part="C12" gate="G$1" x="254" y="-5.08"/>
 <instance part="5V" gate="G$1" x="254" y="7.62" rot="R90"/>
@@
 <instance part="SW_GND1" gate="G$1" x="195.58" y="20.32"/>
 <instance part="SW_GND2" gate="G$1" x="195.58" y="12.7"/>
-<instance part="VCC1" gate="G$1" x="264.16" y="15.24" rot="R90"/>
-<instance part="VCC2" gate="G$1" x="271.78" y="15.24" rot="R90"/>
-<instance part="GND1" gate="G$1" x="264.16" y="-20.32" rot="R270"/>
-<instance part="GND2" gate="G$1" x="274.32" y="-20.32" rot="R270"/>
 <instance part="RST" gate="G$1" x="73.66" y="50.8" rot="R90"/>
 <instance part="RST_GND" gate="G$1" x="50.8" y="50.8" rot="R90"/>
-<instance part="C14" gate="G$1" x="73.66" y="30.48" rot="R180"/>
 <instance part="P2GND" gate="G$1" x="165.1" y="-17.78" rot="R90"/>
 <instance part="P1GND" gate="G$1" x="172.72" y="-17.78" rot="R90"/>
 <instance part="R10" gate="G$1" x="327.66" y="-88.9" rot="R270"/>
+<instance part="C15" gate="G$1" x="205.74" y="7.62" rot="R270"/>
+<instance part="R18" gate="G$1" x="281.94" y="-50.8" rot="R270"/>
 </instances>
 <busses>
@@
 <wire x1="281.94" y1="0" x2="281.94" y2="-12.7" width="0.1524" layer="91"/>
 <junction x="281.94" y="-12.7"/>
-<pinref part="GND1" gate="G$1" pin="1"/>
 <wire x1="264.16" y1="-17.78" x2="264.16" y2="-12.7" width="0.1524" layer="91"/>
 <junction x="264.16" y="-12.7"/>
-<pinref part="GND2" gate="G$1" pin="1"/>
 <wire x1="274.32" y1="-17.78" x2="274.32" y2="-12.7" width="0.1524" layer="91"/>
 <junction x="274.32" y="-12.7"/>
@@
 <pinref part="R17" gate="G$1" pin="2"/>
 <wire x1="254" y1="0" x2="259.08" y2="0" width="0.1524" layer="91"/>
-<pinref part="VCC1" gate="G$1" pin="1"/>
-<wire x1="254" y1="2.54" x2="264.16" y2="2.54" width="0.1524" layer="91"/>
-<wire x1="264.16" y1="2.54" x2="264.16" y2="12.7" width="0.1524" layer="91"/>
+<wire x1="254" y1="2.54" x2="271.78" y2="2.54" width="0.1524" layer="91"/>
 <junction x="254" y="2.54"/>
-<pinref part="VCC2" gate="G$1" pin="1"/>
-<wire x1="264.16" y1="2.54" x2="271.78" y2="2.54" width="0.1524" layer="91"/>
 <wire x1="271.78" y1="2.54" x2="271.78" y2="12.7" width="0.1524" layer="91"/>
-<junction x="264.16" y="2.54"/>
 </segment>
 </net>
@@
 <net name="RESET" class="0">
 <segment>
-<pinref part="JP1" gate="A" pin="1"/>
-<wire x1="203.2" y1="-2.54" x2="190.5" y2="-2.54" width="0.1524" layer="91"/>
-<wire x1="190.5" y1="-2.54" x2="190.5" y2="0" width="0.1524" layer="91"/>
-<label x="190.5" y="0" size="1.778" layer="95"/>
-</segment>
-<segment>
-<pinref part="C14" gate="G$1" pin="2"/>
+<wire x1="208.28" y1="7.62" x2="215.9" y2="7.62" width="0.1524" layer="91"/>
+<label x="213.36" y="5.08" size="1.778" layer="95"/>
+<pinref part="C15" gate="G$1" pin="1"/>
+</segment>
+<segment>
 <pinref part="RST" gate="G$1" pin="1"/>
-<wire x1="73.66" y1="35.56" x2="73.66" y2="48.26" width="0.1524" layer="91"/>
 <label x="73.66" y="38.1" size="1.778" layer="95"/>
+<pinref part="R9" gate="G$1" pin="1"/>
+<pinref part="IC1" gate="G$1" pin="PC6(/RESET)"/>
+<wire x1="71.12" y1="20.32" x2="73.66" y2="20.32" width="0.1524" layer="91"/>
+<wire x1="73.66" y1="20.32" x2="76.2" y2="20.32" width="0.1524" layer="91"/>
+<junction x="73.66" y="20.32"/>
+<label x="71.12" y="17.78" size="1.778" layer="95"/>
+<wire x1="73.66" y1="48.26" x2="73.66" y2="20.32" width="0.1524" layer="91"/>
 </segment>
 </net>
@@
 <segment>
 <label x="281.94" y="-43.18" size="1.778" layer="95"/>
-<wire x1="281.94" y1="-35.56" x2="281.94" y2="-48.26" width="0.1524" layer="91"/>
+<wire x1="281.94" y1="-20.32" x2="281.94" y2="-33.02" width="0.1524" layer="91"/>
 <pinref part="C11" gate="G$1" pin="1"/>
-<junction x="281.94" y="-48.26"/>
+<junction x="281.94" y="-33.02"/>
 </segment>
 </net>
@@
 </segment>
 </net>
-<net name="N$16" class="0">
-<segment>
-<pinref part="C11" gate="G$1" pin="2"/>
-<pinref part="VOLUME" gate="G$1" pin="B"/>
-<wire x1="281.94" y1="-55.88" x2="281.94" y2="-58.42" width="0.1524" layer="91"/>
-</segment>
-</net>
 <net name="N$21" class="0">
 <segment>
@@
 </net>
 <net name="RST0" class="0">
-<segment>
-<pinref part="R9" gate="G$1" pin="1"/>
-<pinref part="IC1" gate="G$1" pin="PC6(/RESET)"/>
-<wire x1="71.12" y1="20.32" x2="73.66" y2="20.32" width="0.1524" layer="91"/>
-<pinref part="C14" gate="G$1" pin="1"/>
-<wire x1="73.66" y1="20.32" x2="76.2" y2="20.32" width="0.1524" layer="91"/>
-<wire x1="73.66" y1="27.94" x2="73.66" y2="20.32" width="0.1524" layer="91"/>
-<junction x="73.66" y="20.32"/>
-<label x="71.12" y="17.78" size="1.778" layer="95"/>
-</segment>
 <segment>
 <label x="134.62" y="-40.64" size="1.778" layer="95"/>
@@
 </segment>
 </net>
+<net name="N$9" class="0">
+<segment>
+<pinref part="C15" gate="G$1" pin="2"/>
+<wire x1="200.66" y1="7.62" x2="190.5" y2="7.62" width="0.1524" layer="91"/>
+<wire x1="190.5" y1="7.62" x2="190.5" y2="-2.54" width="0.1524" layer="91"/>
+<pinref part="JP1" gate="A" pin="1"/>
+<wire x1="190.5" y1="-2.54" x2="203.2" y2="-2.54" width="0.1524" layer="91"/>
+</segment>
+</net>
+<net name="N$16" class="0">
+<segment>
+<pinref part="VOLUME" gate="G$1" pin="B"/>
+<pinref part="R18" gate="G$1" pin="2"/>
+<wire x1="281.94" y1="-58.42" x2="281.94" y2="-55.88" width="0.1524" layer="91"/>
+</segment>
+</net>
+<net name="N$25" class="0">
+<segment>
+<pinref part="R18" gate="G$1" pin="1"/>
+<pinref part="C11" gate="G$1" pin="2"/>
+<wire x1="281.94" y1="-45.72" x2="281.94" y2="-40.64" width="0.1524" layer="91"/>
+</segment>
+</net>

Commit message: add overvoltage protect, refactor
Parts:
- removed 5V, P1GND, P2GND, RST_GND, SPK-, SW_GND1, SW_GND2: (no value), pinhead:PINHD-1X1
- added 5VA, 5VA1, 5VA2, 5VA3, 5VA4, 5VB, GND1, GNDA, GNDB: (no value), pinhead:PINHD-1X1
- added C14: (no value), rcl:C-EUC0805
- added D1: (no value), diode:DIODE-SMC
- added D2: DIODE-ZENER-BZT52, SparkFun:DIODE-ZENER-BZT52
- added PTC1: (no value), microbuilder:PTC1812
- added Q2: NTD5867NL_NMOSFET, jason_eagle6:NTD5867NL_NMOSFET
- added Q3: SCR_BT300S, jason_eagle6:SCR_BT300S
- added R19, R20, R21: (no value), rcl:R-EU_R0805
Connections:
- removed net N$2: IC1.PB4(MISO), ICSP.MISO
- removed net RST0: ICSP.RESET
- new net ENA_STRIP: IC1.PB4(MISO), ICSP.MISO, R21.1
- new net N$28: 5VA.1, 5VB.1, PTC1.2
- new net N$31: C14.1, D2.A, Q3.G, R19.1
- new net N$32: 5VA3.1, 5VA4.1, Q2.D
- new net Z: Q2.G, R20.1, R21.2
- net GND: now also C14.2, D1.A, GND1.1, GNDA.1, GNDB.1, Q2.S, Q3.K, R19.2, R20.2; no longer P1GND.1, P2GND.1, RST_GND.1, SPK-.1, SW_GND1.1, SW_GND2.1
- net RESET: now also ICSP.RESET
- net VCC: now also 5VA1.1, 5VA2.1, D1.C, D2.C, PTC1.1, Q3.A; no longer 5V.1
Other:
- moved on the sheet: GND

Commit message: tweaks
Parts:
- removed 5VA1, 5VA3, 5VB, GNDA: (no value), pinhead:PINHD-1X1
- renumbered 5VA to 5V, GNDB to GND_
Connections:
- net GND: no longer GNDA.1
- net N$28: no longer 5VB.1
- net N$32: no longer 5VA3.1
- net VCC: no longer 5VA1.1
Changed lines of the file:
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@@
 <part name="D2" library="SparkFun" deviceset="DIODE-ZENER" device="-BZT52"/>
 <part name="R19" library="rcl" deviceset="R-EU_" device="R0805"/>
-<part name="5VA" library="pinhead" deviceset="PINHD-1X1" device=""/>
-<part name="5VB" library="pinhead" deviceset="PINHD-1X1" device=""/>
-<part name="GNDA" library="pinhead" deviceset="PINHD-1X1" device=""/>
-<part name="GNDB" library="pinhead" deviceset="PINHD-1X1" device=""/>
+<part name="5V" library="pinhead" deviceset="PINHD-1X1" device=""/>
+<part name="GND_" library="pinhead" deviceset="PINHD-1X1" device=""/>
 <part name="D1" library="diode" deviceset="DIODE-" device="SMC"/>
-<part name="5VA1" library="pinhead" deviceset="PINHD-1X1" device=""/>
 <part name="5VA2" library="pinhead" deviceset="PINHD-1X1" device=""/>
-<part name="5VA3" library="pinhead" deviceset="PINHD-1X1" device=""/>
 <part name="5VA4" library="pinhead" deviceset="PINHD-1X1" device=""/>
 <part name="R20" library="rcl" deviceset="R-EU_" device="R0805"/>
@@
 <instance part="D2" gate="G$1" x="287.02" y="93.98" rot="R90"/>
 <instance part="R19" gate="G$1" x="287.02" y="76.2" rot="R270"/>
-<instance part="5VA" gate="G$1" x="248.92" y="99.06" rot="R180"/>
-<instance part="5VB" gate="G$1" x="248.92" y="93.98" rot="R180"/>
-<instance part="GNDA" gate="G$1" x="248.92" y="73.66" rot="R180"/>
-<instance part="GNDB" gate="G$1" x="248.92" y="68.58" rot="R180"/>
+<instance part="5V" gate="G$1" x="248.92" y="99.06" rot="R180"/>
+<instance part="GND_" gate="G$1" x="248.92" y="68.58" rot="R180"/>
 <instance part="D1" gate="G$1" x="279.4" y="81.28" rot="R90"/>
-<instance part="5VA1" gate="G$1" x="345.44" y="114.3"/>
 <instance part="5VA2" gate="G$1" x="345.44" y="109.22"/>
-<instance part="5VA3" gate="G$1" x="355.6" y="86.36"/>
 <instance part="5VA4" gate="G$1" x="355.6" y="81.28"/>
 <instance part="R20" gate="G$1" x="320.04" y="76.2" rot="R180"/>
@@
 </segment>
 <segment>
-<pinref part="GNDB" gate="G$1" pin="1"/>
+<pinref part="GND_" gate="G$1" pin="1"/>
 <pinref part="Q3" gate="G$1" pin="K"/>
-<wire x1="251.46" y1="68.58" x2="264.16" y2="68.58" width="0.1524" layer="91"/>
-<wire x1="264.16" y1="68.58" x2="279.4" y2="68.58" width="0.1524" layer="91"/>
+<wire x1="251.46" y1="68.58" x2="279.4" y2="68.58" width="0.1524" layer="91"/>
 <wire x1="279.4" y1="68.58" x2="287.02" y2="68.58" width="0.1524" layer="91"/>
 <wire x1="287.02" y1="68.58" x2="297.18" y2="68.58" width="0.1524" layer="91"/>
 <wire x1="297.18" y1="68.58" x2="309.88" y2="68.58" width="0.1524" layer="91"/>
-<pinref part="GNDA" gate="G$1" pin="1"/>
 <wire x1="309.88" y1="68.58" x2="309.88" y2="76.2" width="0.1524" layer="91"/>
 <wire x1="309.88" y1="76.2" x2="309.88" y2="83.82" width="0.1524" layer="91"/>
-<wire x1="251.46" y1="73.66" x2="264.16" y2="73.66" width="0.1524" layer="91"/>
-<wire x1="264.16" y1="73.66" x2="264.16" y2="68.58" width="0.1524" layer="91"/>
-<junction x="264.16" y="68.58"/>
 <pinref part="R19" gate="G$1" pin="2"/>
 <wire x1="287.02" y1="71.12" x2="287.02" y2="68.58" width="0.1524" layer="91"/>
@@
 <wire x1="279.4" y1="83.82" x2="279.4" y2="99.06" width="0.1524" layer="91"/>
 <junction x="279.4" y="99.06"/>
-<pinref part="5VA1" gate="G$1" pin="1"/>
-<wire x1="342.9" y1="114.3" x2="309.88" y2="114.3" width="0.1524" layer="91"/>
-<wire x1="309.88" y1="114.3" x2="309.88" y2="109.22" width="0.1524" layer="91"/>
 <junction x="309.88" y="99.06"/>
 <pinref part="5VA2" gate="G$1" pin="1"/>
 <wire x1="309.88" y1="109.22" x2="309.88" y2="99.06" width="0.1524" layer="91"/>
 <wire x1="342.9" y1="109.22" x2="309.88" y2="109.22" width="0.1524" layer="91"/>
-<junction x="309.88" y="109.22"/>
 <wire x1="309.88" y1="99.06" x2="370.84" y2="99.06" width="0.1524" layer="91"/>
 <label x="370.84" y="99.06" size="1.778" layer="95"/>
@@
 <net name="N$28" class="0">
 <segment>
-<pinref part="5VA" gate="G$1" pin="1"/>
+<pinref part="5V" gate="G$1" pin="1"/>
 <pinref part="PTC1" gate="G$1" pin="2"/>
-<wire x1="251.46" y1="99.06" x2="264.16" y2="99.06" width="0.1524" layer="91"/>
-<pinref part="5VB" gate="G$1" pin="1"/>
-<wire x1="264.16" y1="99.06" x2="266.7" y2="99.06" width="0.1524" layer="91"/>
-<wire x1="251.46" y1="93.98" x2="264.16" y2="93.98" width="0.1524" layer="91"/>
-<wire x1="264.16" y1="93.98" x2="264.16" y2="99.06" width="0.1524" layer="91"/>
-<junction x="264.16" y="99.06"/>
+<wire x1="251.46" y1="99.06" x2="266.7" y2="99.06" width="0.1524" layer="91"/>
 </segment>
 </net>
@@
 <net name="N$32" class="0">
 <segment>
-<pinref part="5VA3" gate="G$1" pin="1"/>
-<wire x1="345.44" y1="81.28" x2="345.44" y2="86.36" width="0.1524" layer="91"/>
-<wire x1="345.44" y1="86.36" x2="353.06" y2="86.36" width="0.1524" layer="91"/>
 <pinref part="5VA4" gate="G$1" pin="1"/>
-<wire x1="353.06" y1="81.28" x2="345.44" y2="81.28" width="0.1524" layer="91"/>
+<wire x1="353.06" y1="81.28" x2="340.36" y2="81.28" width="0.1524" layer="91"/>
 <pinref part="Q2" gate="G$1" pin="D"/>
-<wire x1="340.36" y1="81.28" x2="345.44" y2="81.28" width="0.1524" layer="91"/>
-<junction x="345.44" y="81.28"/>
-</segment>
-</net>
+</segment>
+</net>

Commit message: bits
Parts:
- C11, C14, C9: value (none) -> 100n
- C7: value (none) -> 47n
- R1, R12, R13, R14, R15, R19, R2, R3, R4, R5, R6, R7, R8: value (none) -> 100r
- R10: value (none) -> 10r
- R11, R21: value (none) -> 1k
- R20: value (none) -> 10k
- renumbered R18 to 100K
Changed lines of the file:
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@@
 <part name="U$1" library="jasons_stuff" deviceset="LARGE8X8" device=""/>
 <part name="IC5" library="jasons_stuff" deviceset="NPIC6C596" device=""/>
-<part name="R1" library="rcl" deviceset="R-EU_" device="R0805"/>
-<part name="R2" library="rcl" deviceset="R-EU_" device="R0805"/>
-<part name="R3" library="rcl" deviceset="R-EU_" device="R0805"/>
-<part name="R4" library="rcl" deviceset="R-EU_" device="R0805"/>
-<part name="R5" library="rcl" deviceset="R-EU_" device="R0805"/>
-<part name="R6" library="rcl" deviceset="R-EU_" device="R0805"/>
-<part name="R7" library="rcl" deviceset="R-EU_" device="R0805"/>
-<part name="R8" library="rcl" deviceset="R-EU_" device="R0805"/>
+<part name="R1" library="rcl" deviceset="R-EU_" device="R0805" value="100r"/>
+<part name="R2" library="rcl" deviceset="R-EU_" device="R0805" value="100r"/>
+<part name="R3" library="rcl" deviceset="R-EU_" device="R0805" value="100r"/>
+<part name="R4" library="rcl" deviceset="R-EU_" device="R0805" value="100r"/>
+<part name="R5" library="rcl" deviceset="R-EU_" device="R0805" value="100r"/>
+<part name="R6" library="rcl" deviceset="R-EU_" device="R0805" value="100r"/>
+<part name="R7" library="rcl" deviceset="R-EU_" device="R0805" value="100r"/>
+<part name="R8" library="rcl" deviceset="R-EU_" device="R0805" value="100r"/>
 <part name="U$2" library="jasons_stuff" deviceset="LARGE8X8" device=""/>
 <part name="IC4" library="jasons_stuff" deviceset="NPIC6C596" device=""/>
@@
 <part name="JP1" library="pinhead" deviceset="PINHD-1X6" device=""/>
 <part name="IC2" library="74xx-eu" deviceset="74*257" device="D" technology="HC"/>
-<part name="R12" library="rcl" deviceset="R-EU_" device="R0805"/>
-<part name="R13" library="rcl" deviceset="R-EU_" device="R0805"/>
-<part name="R14" library="rcl" deviceset="R-EU_" device="R0805"/>
-<part name="R15" library="rcl" deviceset="R-EU_" device="R0805"/>
+<part name="R12" library="rcl" deviceset="R-EU_" device="R0805" value="100r"/>
+<part name="R13" library="rcl" deviceset="R-EU_" device="R0805" value="100r"/>
+<part name="R14" library="rcl" deviceset="R-EU_" device="R0805" value="100r"/>
+<part name="R15" library="rcl" deviceset="R-EU_" device="R0805" value="100r"/>
 <part name="MOSI1" library="pinhead" deviceset="PINHD-1X1" device=""/>
 <part name="MOSI2" library="pinhead" deviceset="PINHD-1X1" device=""/>
@@
 <part name="IC3" library="linear" deviceset="LM386?-*" device="M" technology="1"/>
 <part name="SPK+" library="pinhead" deviceset="PINHD-1X1" device=""/>
-<part name="C7" library="rcl" deviceset="C-EU" device="C0805"/>
+<part name="C7" library="rcl" deviceset="C-EU" device="C0805" value="47n"/>
 <part name="C8" library="rcl" deviceset="CPOL-EU" device="E2.5-6"/>
 <part name="C10" library="rcl" deviceset="C-EU" device="C0805"/>
 <part name="R16" library="rcl" deviceset="R-EU_" device="R0805"/>
-<part name="C11" library="rcl" deviceset="C-EU" device="C0805"/>
+<part name="C11" library="rcl" deviceset="C-EU" device="C0805" value="100n"/>
 <part name="C12" library="rcl" deviceset="CPOL-EU" device="E2.5-6"/>
 <part name="PWR" library="adafruit" deviceset="LED" device="3MM"/>
 <part name="R17" library="rcl" deviceset="R-EU_" device="R0805"/>
 <part name="DIAG" library="adafruit" deviceset="LED" device="3MM"/>
-<part name="R11" library="rcl" deviceset="R-EU_" device="R0805"/>
+<part name="R11" library="rcl" deviceset="R-EU_" device="R0805" value="1k"/>
 <part name="VOLUME" library="jasons_stuff" deviceset="ALPS_POT_SMALL" device=""/>
 <part name="C13" library="rcl" deviceset="CPOL-EU" device="E2.5-6"/>
-<part name="C9" library="rcl" deviceset="C-EU" device="C0805"/>
+<part name="C9" library="rcl" deviceset="C-EU" device="C0805" value="100n"/>
 <part name="ICSP" library="jasons_stuff" deviceset="TAG_CONN_AVR" device=""/>
 <part name="RST" library="pinhead" deviceset="PINHD-1X1" device=""/>
-<part name="R10" library="rcl" deviceset="R-EU_" device="R0805"/>
+<part name="R10" library="rcl" deviceset="R-EU_" device="R0805" value="10r"/>
 <part name="C15" library="rcl" deviceset="C-EU" device="C0805"/>
-<part name="R18" library="rcl" deviceset="R-EU_" device="R0805"/>
+<part name="100K" library="rcl" deviceset="R-EU_" device="R0805"/>
 <part name="Q3" library="jason_eagle6" deviceset="SCR_BT300S" device=""/>
 <part name="PTC1" library="microbuilder" deviceset="PTC" device="1812"/>
 <part name="D2" library="SparkFun" deviceset="DIODE-ZENER" device="-BZT52"/>
-<part name="R19" library="rcl" deviceset="R-EU_" device="R0805"/>
+<part name="R19" library="rcl" deviceset="R-EU_" device="R0805" value="100r"/>
 <part name="5V" library="pinhead" deviceset="PINHD-1X1" device=""/>
 <part name="GND_" library="pinhead" deviceset="PINHD-1X1" device=""/>
@@
 <part name="5VA2" library="pinhead" deviceset="PINHD-1X1" device=""/>
 <part name="5VA4" library="pinhead" deviceset="PINHD-1X1" device=""/>
-<part name="R20" library="rcl" deviceset="R-EU_" device="R0805"/>
-<part name="C14" library="rcl" deviceset="C-EU" device="C0805"/>
+<part name="R20" library="rcl" deviceset="R-EU_" device="R0805" value="10k"/>
+<part name="C14" library="rcl" deviceset="C-EU" device="C0805" value="100n"/>
 <part name="Q2" library="jason_eagle6" deviceset="NTD5867NL_NMOSFET" device=""/>
-<part name="R21" library="rcl" deviceset="R-EU_" device="R0805"/>
+<part name="R21" library="rcl" deviceset="R-EU_" device="R0805" value="1k"/>
 <part name="GND" library="pinhead" deviceset="PINHD-1X1" device=""/>
 <part name="GND1" library="pinhead" deviceset="PINHD-1X1" device=""/>
@@
 <instance part="R10" gate="G$1" x="327.66" y="-88.9" rot="R270"/>
 <instance part="C15" gate="G$1" x="205.74" y="7.62" rot="R270"/>
-<instance part="R18" gate="G$1" x="281.94" y="-50.8" rot="R270"/>
+<instance part="100K" gate="G$1" x="281.94" y="-50.8" rot="R270"/>
 <instance part="Q3" gate="G$1" x="309.88" y="91.44" rot="R270"/>
 <instance part="PTC1" gate="G$1" x="271.78" y="99.06"/>
@@
 <segment>
 <pinref part="VOLUME" gate="G$1" pin="B"/>
-<pinref part="R18" gate="G$1" pin="2"/>
+<pinref part="100K" gate="G$1" pin="2"/>
 <wire x1="281.94" y1="-58.42" x2="281.94" y2="-55.88" width="0.1524" layer="91"/>
 </segment>
@@
 <net name="N$25" class="0">
 <segment>
-<pinref part="R18" gate="G$1" pin="1"/>
+<pinref part="100K" gate="G$1" pin="1"/>
 <pinref part="C11" gate="G$1" pin="2"/>
 <wire x1="281.94" y1="-45.72" x2="281.94" y2="-40.64" width="0.1524" layer="91"/>

Commit message: tidy up values
Parts:
- renumbered 100K to R18
Changed lines of the file:
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@@
 <part name="R10" library="rcl" deviceset="R-EU_" device="R0805" value="10r"/>
 <part name="C15" library="rcl" deviceset="C-EU" device="C0805"/>
-<part name="100K" library="rcl" deviceset="R-EU_" device="R0805"/>
+<part name="R18" library="rcl" deviceset="R-EU_" device="R0805"/>
 <part name="Q3" library="jason_eagle6" deviceset="SCR_BT300S" device=""/>
 <part name="PTC1" library="microbuilder" deviceset="PTC" device="1812"/>
@@
 <instance part="R10" gate="G$1" x="327.66" y="-88.9" rot="R270"/>
 <instance part="C15" gate="G$1" x="205.74" y="7.62" rot="R270"/>
-<instance part="100K" gate="G$1" x="281.94" y="-50.8" rot="R270"/>
+<instance part="R18" gate="G$1" x="281.94" y="-50.8" rot="R270"/>
 <instance part="Q3" gate="G$1" x="309.88" y="91.44" rot="R270"/>
 <instance part="PTC1" gate="G$1" x="271.78" y="99.06"/>
@@
 <segment>
 <pinref part="VOLUME" gate="G$1" pin="B"/>
-<pinref part="100K" gate="G$1" pin="2"/>
+<pinref part="R18" gate="G$1" pin="2"/>
 <wire x1="281.94" y1="-58.42" x2="281.94" y2="-55.88" width="0.1524" layer="91"/>
 </segment>
@@
 <net name="N$25" class="0">
 <segment>
-<pinref part="100K" gate="G$1" pin="1"/>
+<pinref part="R18" gate="G$1" pin="1"/>
 <pinref part="C11" gate="G$1" pin="2"/>
 <wire x1="281.94" y1="-45.72" x2="281.94" y2="-40.64" width="0.1524" layer="91"/>

Commit message: poss V3
Parts:
- removed D2: DIODE-ZENER-BZT52, SparkFun:DIODE-ZENER-BZT52
- removed Q3: SCR_BT300S, jason_eagle6:SCR_BT300S
- removed R19: 100r, rcl:R-EU_R0805
- added C16: 1u, rcl:C-EUC0805
- added IC6: NCP361SNT1G, jason_eagle6:NCP361SNT1G
- added R22: 100r, rcl:R-EU_R0805
- added TP2: TPB2,54, testpad:TPB2,54
- C14: value 100n -> 1u
Connections:
- removed net N$13: IC1.PB2(SS/OC1B), IC2A.!A!/B
- removed net N$31: C14.1, D2.A, Q3.G, R19.1
- new net MISO: IC1.PB4(MISO), ICSP.MISO
- new net N$2: IC2A.!A!/B, R22.1
- new net VIN: 5VA2.1, C14.1, D1.C, IC6.IN, PTC1.1
- net ENA_STRIP: now also IC1.PB2(SS/OC1B), TP2.TP; no longer IC1.PB4(MISO), ICSP.MISO
- net GND: now also C16.2, IC6.EN#, IC6.GND, R22.2; no longer Q3.K, R19.2
- net VCC: now also C16.1, IC6.OUT; no longer 5VA2.1, D1.C, D2.C, PTC1.1, Q3.A
Other:
- moved on the sheet: 5VA2, 5VA4, C14, Q2, R20, R21
