File: oneDpong.sch (EAGLE design)
At the start: 72 parts, among them IC1 NPIC6C596, IC2 74HC257D, IC3 MEGA8-AI, IC4 LM386M-1, IC5 NPIC6C596, IC6 NCP361SNT1G, Q1 SPD30P06PTO252

Commit message: updates
Parts:
- C11, R15: value (none) -> DNF
- R14: value (none) -> 4k7
Other:
- note added: "10KA"
Changed lines of the file:
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@@
 <part name="C10" library="rcl" deviceset="C-EU" device="C0805" value="47n"/>
 <part name="C8" library="rcl" deviceset="CPOL-EU" device="E2.5-6"/>
-<part name="C11" library="rcl" deviceset="C-EU" device="C0805"/>
-<part name="R15" library="rcl" deviceset="R-EU_" device="R0805"/>
+<part name="C11" library="rcl" deviceset="C-EU" device="C0805" value="DNF"/>
+<part name="R15" library="rcl" deviceset="R-EU_" device="R0805" value="DNF"/>
 <part name="C13" library="rcl" deviceset="C-EU" device="C0805" value="100n"/>
 <part name="C9" library="rcl" deviceset="CPOL-EU" device="E2.5-6"/>
@@
 <part name="R13" library="rcl" deviceset="R-EU_" device="R0805" value="10r"/>
 <part name="C1" library="rcl" deviceset="C-EU" device="C0805"/>
-<part name="R14" library="rcl" deviceset="R-EU_" device="R0805"/>
+<part name="R14" library="rcl" deviceset="R-EU_" device="R0805" value="4k7"/>
 <part name="PTC1" library="microbuilder" deviceset="PTC" device="1812"/>
 <part name="5V" library="pinhead" deviceset="PINHD-1X1" device=""/>
@@
 <sheet>
 <plain>
+<text x="284.48" y="-76.2" size="1.778" layer="91">10KA</text>
 </plain>
 <instances>
